Commit message: replaced topics to match oxts driver instead of imu preintegration

File: launch/include/config/robot.astarig.xacro (robot description, xacro)
@@ -9,8 +9,8 @@
     <origin xyz="0 0 0" rpy="0 0 0" />
   </joint>
-  <link name="OxTs"> </link>
+  <link name="oxts_link"> </link>
   <joint name="imu_joint" type="fixed">
     <parent link="base_link" />
-    <child link="OxTs"/>
+    <child link="oxts_link"/>
     <origin xyz="0 0 0" rpy="0 0 0" />
   </joint>
@@ -23,5 +23,5 @@
   <link name="navsat_link"> </link>
   <joint name="navsat_joint" type="fixed">
-    <parent link="OxTs" />
+    <parent link="oxts_link" />
     <child link="navsat_link" />
     <origin xyz="0 0 0" rpy="0 0 0" />

Commit message: Moved some stuff to OxTs decoder and this no longe rstarts ImuPreintegration node

File: launch/include/config/robot.astarig.xacro (robot description, xacro)
@@ -9,21 +9,9 @@
     <origin xyz="0 0 0" rpy="0 0 0" />
   </joint>
-  <link name="oxts_link"> </link>
-  <joint name="imu_joint" type="fixed">
-    <parent link="base_link" />
-    <child link="oxts_link"/>
-    <origin xyz="0 0 0" rpy="0 0 0" />
-  </joint>
   <link name="velodyne"> </link>
   <joint name="velodyne_joint" type="fixed">
     <parent link="chassis_link"/>
     <child link="velodyne" />
-    <origin xyz="0.0 0.0 0.246" rpy="0 0 0" />
-  </joint>
-  <link name="navsat_link"> </link>
-  <joint name="navsat_joint" type="fixed">
-    <parent link="oxts_link" />
-    <child link="navsat_link" />
-    <origin xyz="0 0 0" rpy="0 0 0" />
+    <origin xyz="0.681 0.0 0.813" rpy="0 0 0" />
   </joint>
 </robot>
