Commit message: kinda working

File: config/robot.astarig.xacro (robot description, xacro)
@@ -9,8 +9,8 @@
     <origin xyz="0 0 0" rpy="0 0 0" />
   </joint>
-  <link name="oxts_link"> </link>
+  <link name="imu_link"> </link>
   <joint name="imu_joint" type="fixed">
     <parent link="base_link" />
-    <child link="oxts_link"/>
+    <child link="imu_link"/>
     <origin xyz="0 0 0" rpy="0 0 0" />
   </joint>
@@ -23,5 +23,5 @@
   <link name="navsat_link"> </link>
   <joint name="navsat_joint" type="fixed">
-    <parent link="oxts_link" />
+    <parent link="imu_link" />
     <child link="navsat_link" />
     <origin xyz="0 0 0" rpy="0 0 0" />
